File: PCB_Sch_v1.sch (EAGLE design)
At the start: 0 parts

Commit message: Added libraries and v1
Parts:
- added U1: ESP32-WROOM-32D, ESP32-WROOM-32D:ESP32-WROOM-32D
Changed lines of the file:
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@@
 </classes>
 <parts>
+<part name="U1" library="ESP32-WROOM-32D" deviceset="ESP32-WROOM-32D" device=""/>
 </parts>
 <sheets>
@@
 </plain>
 <instances>
+<instance part="U1" gate="G$1" x="81.28" y="38.1" smashed="yes">
+<attribute name="NAME" x="66.2441" y="74.7745" size="1.783840625" layer="95"/>
+<attribute name="VALUE" x="65.9933" y="-0.1081" size="1.78345" layer="96"/>
+</instance>
 </instances>
 <busses>
