File: PCB_Sch_v3.sch (EAGLE design)
At the start: 38 parts, among them J1 10118193-0001LF, M1 C0720B001F, Q3 DMG3415U, SW2 2-1825027-0, SW3 2-1825027-0, SW4 2-1825027-0, SW5 2-1825027-0, T1 2N2222, U1 ESP32-WROOM-32D, U2 UG-2828GDEDF11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

Commit message: Added other parts, organized, changed some of the I/O pins
Parts:
- removed J1: 10118193-0001LF, 10118193-0001LF:10118193-0001LF
- removed R2, R3, R6, R7, R8: 100K, adafruit:R-US_R0805
- removed T1: 2N2222, adafruit:2N2222
- added C11: 10uF, microbuilder:CAP_CERAMIC0805
- added C12: 0.1uF, microbuilder:CAP_CERAMIC0805
- added C14: 0.1uF, SparkFun-Capacitors:0.1UF-0603-25V-(+80/-20%)
- added D5: BAT54T1G, microbuilder:DIODESOD-123
- added IC1: CP2104, microbuilder:CP2104
- added L1: 10uH, microbuilder:INDUCTOR
- added Q1: MMBT2222LT1G, MMBT2222LT1G:MMBT2222LT1G
- added Q2, Q4: mmbt2222, SparkFun:TRANSISTOR_NPNSOT23-3
- added R11: 100K, microbuilder:RESISTOR0805
- added R12: 10K, microbuilder:RESISTOR0805
- added SW1: 2-1825027-0, 2-1825027-0:2-1825027-0
- added U5: FAN5331SX, microbuilder:FAN5331
- added X4: 20329, microbuilder:USB_MICRO_20329_V2
- U3: value AP2112K-3.3TRG1 -> MCP73831T-2ACI/OT; device AP2112K-3.3TRG1:AP2112K-3.3TRG1 -> microbuilder:MCP73831/2
Connections:
- net N$9 renamed MOTOR
- removed net B0: R2.2, U1.IO25
- removed net B1: R6.2, SW2.1, U1.IO34
- removed net B2: R7.2, SW3.1, U1.SENSOR_VN
- removed net B3: R8.2, SW4.1, U1.SENSOR_VP
- removed net D-OUT: MK1.DATA_OUT, U1.IO12
- removed net LRC: MK1.WS, U1.TXD0
- removed net N$10: MK1.BCLK, U1.RXD0
- removed net N$15: Q3.D
- new net 3.3V1: C14.1, IC1G$1.REGIN, IC1G$1.VDD, IC1G$1.VIO
- new net BTN_LL: U1.IO12
- new net BTN_LR: U1.IO0
- new net BTN_UL: U1.IO34
- new net BTN_UR: U1.IO23
- new net BTN_WRIST: U1.IO2
- new net DTR: IC1G$1.DTR
- new net DTR1: Q4.E
- new net GPIO0: Q4.C
- new net I2S_BCLK: MK1.BCLK, U1.IO14
- new net I2S_DOUT: MK1.DATA_OUT, U1.IO32
- new net I2S_LRCLK: MK1.WS, U1.IO15
- new net N$13: D5.A, L1.2, U5.SW
- new net N$16: C12.P$2, R11.1, R12.2, U5.FB
- new net N$9: Q4.B
- new net OLED_MOSI: U1.IO18
- new net OLED_RST: U1.IO17
- new net RESET: Q2.C
- new net RTS: IC1G$1.RTS
- new net RTS1: Q2.E
- new net RXD0: IC1G$1.TXD
- new net SCK: U1.IO5
- new net TXD0: IC1G$1.RXD
- new net VBUS1: IC1G$1.VBUS, X4.VBUS
- net 13V: now also C12.P$1, D5.C, R11.2
- net 3.3V: now also C11.P$1, C6.1, D2.C, L1.1, M1.V+, U1.3V3, U5.SHDN, U5.VIN
- net B4: no longer R3.2, SW5.1
- net GND: now also C11.P$2, C14.2, IC1G$1.GND, IC1G$2.TP, Q1.E, R12.1, U5.GND, X4.GND
- net N$1: now also IC1G$1.D+, X4.D+; no longer C6.1, D2.C, M1.V+, T1.C
- net N$2: now also Q1.B; no longer T1.B
- net N$4: now also Q1.C
- net N$5: now also IC1G$1.D-, X4.D-; no longer MK1.VDD, SW2.2, SW3.2, SW4.2, SW5.2
- net N$8: now also Q2.B; no longer R2.1, R3.1, R6.1, R7.1, R8.1
- net OLED_CS: now also U1.IO21
- net OLED_DC: now also U1.IO19
- net VBAT: now also Q3.D
Other:
- note added: "13V Boost"
- note added: "This is 0.5V above the recommended voltage,"
- note added: "USB TO SERIAL CONVERTER"
- note added: "VOUT = 1.23V * (1 + R6/R7)"
- note added: "VOUT = 13.53V"
- note added: "but uses common resistors for easy assembly"
