File: PCB_Sch_v4.sch (EAGLE design)
At the start: 51 parts, among them IC1 CP2104, M1 C0720B001F, Q1 MMBT2222LT1G, Q2 mmbt2222, Q3 DMG3415U, Q4 mmbt2222, SW1 2-1825027-0, SW2 2-1825027-0, SW3 2-1825027-0, SW4 2-1825027-0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

Commit message: Add files via upload
Parts:
- removed C1, C2: 10uF/16V, microbuilder:CAP_CERAMIC0805
- removed C3: 1.0uF, microbuilder:CAP_CERAMIC0805
- removed R12: 10K, microbuilder:RESISTOR0805
- removed R4: 600K, microbuilder:RESISTOR0805
- added C14: 0.1uF, rcl:C-USC0603
- added C16: 10uF/16V, rcl:C-USC0603
- added C17: 1uF, rcl:C-USC0603
- added R13: 10k, rcl:R-US_R0603
- added R8: 100k, rcl:R-US_R0603
- C10, C7, C8, C9: device adafruit:C-USC0805 -> rcl:C-USC0603
- C11: device microbuilder:CAP_CERAMIC0805 -> rcl:C-USC0603
- C12: value 0.1uF -> 10uF; device microbuilder:CAP_CERAMIC0805 -> rcl:C-USC0603
- C4: value 1.0uF -> 10uF/16V; device microbuilder:CAP_CERAMIC0805 -> rcl:C-USC0603
- C5: value 10uF -> 1uF; device microbuilder:CAP_CERAMIC0805 -> rcl:C-USC0603
- C6: value (none) -> 0.1uF; device adafruit:C-USC0805 -> rcl:C-USC0603
- R1: value 1k -> 50; device adafruit:R-US_R0805 -> rcl:R-US_R0603
- R10, R9: device adafruit:R-US_R0805 -> rcl:R-US_R0603
- R11: value 100K -> 1k; device microbuilder:RESISTOR0805 -> rcl:R-US_R0603
- R5: value 50 -> 600k; device microbuilder:RESISTOR0805 -> rcl:R-US_R0603
Connections:
- removed net 3.3V1: C13.1, IC1G$1.REGIN, IC1G$1.VDD, IC1G$1.VIO
- removed net IREF: R4.2, U2.IREF
- removed net VCOMH: C2.P$1, U2.VCOMH
- new net N$18: C16.2, U2.VCOMH
- new net N$19: R5.2, U2.IREF
- net 13V: now also C14.1, C4.1, R10.2; no longer C1.P$2, C12.P$1, R11.2
- net 3.3V: now also C11.2, C12.1, C13.1, C17.1, IC1G$1.REGIN, IC1G$1.VDD, IC1G$1.VIO; no longer C11.P$1, C3.P$2, C5.P$1
- net GND: now also C11.1, C12.2, C16.1, C17.2, C4.2, C5.1, R13.1, R5.1, R8.1; no longer C1.P$1, C11.P$2, C2.P$2, C3.P$1, C4.P$2, C5.P$2, R12.1, R4.1, R9.1
- net MOTOR: now also R11.2; no longer R1.1
- net N$12: now also R9.2; no longer R10.2
- net N$14: now also R9.1; no longer R10.1
- net N$16: now also C14.2, R10.1, R13.2; no longer C12.P$2, R11.1, R12.2
- net N$2: now also R11.1; no longer R1.2
- net N$3: now also C5.2; no longer C4.P$1
- net N$6: now also D1.A, R1.1; no longer R5.2, U2.VSL
- net N$7: now also R1.2, U2.VSL; no longer D1.A, R5.1
- net VBUS: now also R8.2; no longer R9.2
Other:
- moved on the sheet: C11, C12, C4, C5, R1, R10, R9

Commit message: Add files via upload
Parts:
- added M2: C0720B001F, C0720B001F:C0720B001F
Connections:
- new net N$20: M1.V-, M2.V+
- net N$4: now also M2.V-; no longer M1.V-
Other:
- moved on the sheet: C6, D2, M1, Q1, R11, SW1, SW2, SW3, SW4, SW5
