File: PCB_Sch_v6.brd (EAGLE design)
At the start: 38.3 x 38.1 mm, 60 parts, among them IC1 CP2104, M1 C0720B001F, Q1 MMBT2222LT1G, Q2 mmbt2222, Q3 DMG3415U, Q4 mmbt2222, U1 ESP32-WROOM-32D, U2 UG-2828GDEDF11, U3 MCP73831T-2ACI/OT, U4 AP2112-3.3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

Commit message: Progress made on 03/25/2019
Parts:
- moved R6 102.8 mm to (30.0, 14.0)
- moved C13 96.7 mm to (25.4, 17.5), turned to 90 degrees
- moved C15 93.2 mm to (17.5, 22.9)
- moved C9 85.2 mm to (21.3, 25.4), turned to 90 degrees
- moved CHG 84.3 mm to (22.4, 19.1)
- moved D4 71.5 mm to (29.2, 22.1)
- moved R8 68.8 mm to (25.4, 21.6), turned to 90 degrees
- moved R3 65.8 mm to (17.0, 15.2)
- moved R2 65.0 mm to (20.1, 19.1), turned to 90 degrees
- moved C10 26.4 mm to (22.6, 28.7)
- moved R15 23.3 mm to (2.79, 12.4)
- moved Q1 19.0 mm to (6.35, 17.5)
- moved S5 10.8 mm to (8.38, 3.30)
- moved Q3 10.3 mm to (33.3, 25.7), turned to 270 degrees
- moved C7 9.25 mm to (36.6, 25.4)
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
Commit message: Update PCB_Sch_v6.brd
Parts:
- moved U2 64.0 mm to (18.3, 4.32)
- moved S5 22.9 mm to (4.57, 25.9)
- moved L1 22.2 mm to (10.9, 19.6)
- moved R12 5.68 mm to (2.54, 8.89)
