File: PCB_Sch_v8.sch (EAGLE design)
At the start: 60 parts, among them IC1 CP2104, M1 C0720B001F, Q1 MMBT2222LT1G, Q2 mmbt2222, Q3 DMG3415U, Q4 mmbt2222, U1 ESP32-WROOM-32D, U2 UG-2828GDEDF11, U3 MCP73831T-2ACI/OT, U4 AP2112-3.3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

Commit message: Started routing, made some fixes
Connections:
- removed net OUT: C8.1, C9.1, U4.OUT
- net 3.3V: now also C8.1, C9.1, U4.OUT
Changed lines of the file:
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@@
 <pinref part="S5" gate="G$1" pin="4"/>
+</segment>
+<segment>
+<pinref part="U4" gate="G$1" pin="OUT"/>
+<wire x1="-17.78" y1="63.5" x2="-15.24" y2="63.5" width="0.1524" layer="91"/>
+<pinref part="U$13" gate="G$1" pin="3.3V"/>
+<wire x1="-15.24" y1="63.5" x2="-7.62" y2="63.5" width="0.1524" layer="91"/>
+<wire x1="-7.62" y1="63.5" x2="-7.62" y2="78.74" width="0.1524" layer="91"/>
+<pinref part="C9" gate="G$1" pin="1"/>
+<wire x1="-7.62" y1="63.5" x2="-7.62" y2="55.88" width="0.1524" layer="91"/>
+<junction x="-7.62" y="63.5"/>
+<pinref part="C8" gate="G$1" pin="1"/>
+<wire x1="-15.24" y1="63.5" x2="-15.24" y2="55.88" width="0.1524" layer="91"/>
+<junction x="-15.24" y="63.5"/>
 </segment>
 </net>
@@
 </segment>
 </net>
-<net name="OUT" class="0">
-<segment>
-<pinref part="U4" gate="G$1" pin="OUT"/>
-<wire x1="-17.78" y1="63.5" x2="-15.24" y2="63.5" width="0.1524" layer="91"/>
-<wire x1="-15.24" y1="63.5" x2="-7.62" y2="63.5" width="0.1524" layer="91"/>
-<wire x1="-7.62" y1="55.88" x2="-7.62" y2="63.5" width="0.1524" layer="91"/>
-<wire x1="-15.24" y1="55.88" x2="-15.24" y2="63.5" width="0.1524" layer="91"/>
-<junction x="-15.24" y="63.5"/>
-<junction x="-7.62" y="63.5"/>
-<wire x1="-7.62" y1="78.74" x2="-7.62" y2="63.5" width="0.1524" layer="91"/>
-<pinref part="U$13" gate="G$1" pin="3.3V"/>
-<pinref part="C8" gate="G$1" pin="1"/>
-<pinref part="C9" gate="G$1" pin="1"/>
-</segment>
-</net>

Commit message: Final design
Parts:
- removed S5: 434333045822, 434333045822:434333045822
Connections:
- net 3.3V: no longer S5.4
- net BTN_WRIST: no longer R16.2, S5.1
Changed lines of the file:
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@@
 <part name="S3" library="434333045822" deviceset="434333045822" device=""/>
 <part name="S4" library="434333045822" deviceset="434333045822" device=""/>
-<part name="S5" library="434333045822" deviceset="434333045822" device=""/>
 <part name="C3" library="rcl" library_urn="urn:adsk.eagle:library:334" deviceset="C-US" device="C0603" package3d_urn="urn:adsk.eagle:package:23616/2" value="10uF"/>
 <part name="U$40" library="microbuilder" deviceset="GND" device=""/>
@@
 <part name="U$48" library="microbuilder" deviceset="3.3V" device=""/>
 <part name="U$49" library="microbuilder" deviceset="3.3V" device=""/>
-<part name="U$50" library="microbuilder" deviceset="3.3V" device=""/>
 <part name="U$51" library="microbuilder" deviceset="3.3V" device=""/>
 <part name="R17" library="rcl" library_urn="urn:adsk.eagle:library:334" deviceset="R-US_" device="R0603" package3d_urn="urn:adsk.eagle:package:23555/2" value="10k"/>
@@
 <attribute name="VALUE" x="78.74098125" y="128.27146875" size="1.778690625" layer="96" rot="R90"/>
 </instance>
-<instance part="S5" gate="G$1" x="104.14" y="124.46" smashed="yes" rot="R90">
-<attribute name="NAME" x="102.86951875" y="128.27143125" size="1.77866875" layer="95" rot="R90"/>
-<attribute name="VALUE" x="106.68098125" y="128.27146875" size="1.778690625" layer="96" rot="R90"/>
-</instance>
 <instance part="C3" gate="G$1" x="91.44" y="88.9" smashed="yes">
 <attribute name="NAME" x="92.456" y="89.535" size="1.778" layer="95"/>
@@
 <instance part="U$49" gate="G$1" x="86.36" y="129.54" smashed="yes" rot="R270">
 <attribute name="VALUE" x="87.376" y="131.064" size="1.27" layer="96" rot="R270"/>
-</instance>
-<instance part="U$50" gate="G$1" x="114.3" y="129.54" smashed="yes" rot="R270">
-<attribute name="VALUE" x="115.316" y="131.064" size="1.27" layer="96" rot="R270"/>
 </instance>
 <instance part="U$51" gate="G$1" x="66.04" y="-2.54" smashed="yes" rot="R270">
@@
 </segment>
 <segment>
-<pinref part="U$50" gate="G$1" pin="3.3V"/>
-<wire x1="111.76" y1="129.54" x2="109.22" y2="129.54" width="0.1524" layer="91"/>
-<pinref part="S5" gate="G$1" pin="4"/>
-</segment>
-<segment>
 <pinref part="U4" gate="G$1" pin="OUT"/>
 <wire x1="-17.78" y1="63.5" x2="-15.24" y2="63.5" width="0.1524" layer="91"/>
@@
 <label x="58.42" y="71.12" size="1.778" layer="95"/>
 </segment>
-<segment>
-<pinref part="S5" gate="G$1" pin="1"/>
-<wire x1="99.06" y1="119.38" x2="99.06" y2="116.84" width="0.1524" layer="91"/>
-<wire x1="99.06" y1="116.84" x2="93.98" y2="116.84" width="0.1524" layer="91"/>
-<pinref part="R16" gate="G$1" pin="2"/>
-<junction x="99.06" y="116.84"/>
-<label x="83.82" y="116.84" size="1.778" layer="95"/>
-</segment>
-</net>
+</net>
